Commit message: revert to old wire frame

File: penta_description/urdf/wire_frame.urdf.xacro (robot description, xacro)
@@ -1,14 +1,11 @@
 <?xml version="1.0"?>
 <robot name="penta_bot" xmlns:xacro="http://www.ros.org/wiki/xacro">
-  <xacro:property name="PI" value="3.141592" />
-  <xacro:property name="PI2" value="${PI/2}" />
-  <xacro:property name="base_visual_yaw" value="0.32" />
   <link name="base_footprint"/>
   <link name="base_link">
     <visual>
       <geometry>
-        <mesh filename="package://penta_description/meshes/visual/penta_stl_v1/Chassi_middle.stl" scale="0.001 0.001 0.001"/>
+        <cylinder radius="0.085" length="0.025"/>
       </geometry>
-      <origin xyz="0.0 0.0 0.0" rpy="0 0 ${base_visual_yaw}"/>
+      <origin xyz="0.0 0.0 0.0" rpy="0 0 0"/>
     </visual>
   </link>
@@ -21,5 +18,5 @@
     <visual>
       <geometry>
-        <sphere radius="0.01"/>
+        <sphere radius="0.05"/>
       </geometry>
       <material name="green">
@@ -33,20 +30,5 @@
     <origin xyz="-0.1 0.0 0.025" rpy="0 0 0"/>
   </joint>
-  <xacro:macro name="add_base_plate" params="name stl_file_name z">
-    <link name="${name}_link">
-      <visual>
-        <geometry>
-          <mesh filename="package://penta_description/meshes/visual/penta_stl_v1/${stl_file_name}" scale="0.001 0.001 0.001"/>
-        </geometry>
-        <origin xyz="0.0 0.0 0.0" rpy="0 0 ${base_visual_yaw}"/>
-      </visual>
-    </link>
-    <joint name="${name}_joint" type="fixed">
-      <parent link="base_link"/>
-      <child link="${name}_link"/>
-    <origin xyz="0.0 0.0 ${z}" rpy="0 0 0"/>
-  </joint>
-  </xacro:macro>
-  <xacro:macro name="add_leg" params="prefix shoulderxyz shoulderrpy">
+  <xacro:macro name="leg" params="prefix shoulderxyz shoulderrpy">
     <link name="${prefix}_shoulder_motor">
       <visual>
@@ -60,7 +42,7 @@
       <visual>
         <geometry>
-          <mesh filename="package://penta_description/meshes/visual/penta_stl_v1/Shoulder.stl" scale="0.001 0.001 0.001"/>
+          <box size="0.0455 0.02 0.02"/>
         </geometry>
-        <origin xyz="0.0 0.0 0.0" rpy="-${PI2} 0 0"/>
+        <origin xyz="0.02275 0.0 0.0" rpy="0 0 0"/>
       </visual>
     </link>
@@ -68,7 +50,7 @@
       <visual>
         <geometry>
-          <mesh filename="package://penta_description/meshes/visual/penta_stl_v1/Upper_arm.stl" scale="0.001 0.001 0.001"/>
+          <box size="0.096 0.02 0.02"/>
         </geometry>
-        <origin xyz="0.0 0.0 0.0" rpy="0 0 0"/>
+        <origin xyz="0.048 0.0 0.0" rpy="0 0 0"/>
       </visual>
     </link>
@@ -76,7 +58,7 @@
       <visual>
         <geometry>
-          <mesh filename="package://penta_description/meshes/visual/penta_stl_v1/Lower_arm.stl" scale="0.001 0.001 0.001"/>
+          <box size="0.158 0.02 0.02"/>
         </geometry>
-        <origin xyz="0.0 0.0 0.0" rpy="-${PI2} ${PI2} 0.4"/>
+        <origin xyz="0.079 0.0 0.0" rpy="0 0 0"/>
       </visual>
     </link>
@@ -105,10 +87,8 @@
     </joint>
   </xacro:macro>
-<xacro:add_leg prefix="limb0" shoulderxyz="${0.085*cos(0.*3.141592/2.5)} ${0.085*sin(0.*3.141592/2.5)} 0." shoulderrpy="0. 0. ${(0.*3.141592/2.5)}"/>
-<xacro:add_leg prefix="limb1" shoulderxyz="${0.085*cos(1.*3.141592/2.5)} ${0.085*sin(1.*3.141592/2.5)} 0." shoulderrpy="0. 0. ${(1.*3.141592/2.5)}"/>
-<xacro:add_leg prefix="limb2" shoulderxyz="${0.085*cos(2.*3.141592/2.5)} ${0.085*sin(2.*3.141592/2.5)} 0." shoulderrpy="0. 0. ${(2.*3.141592/2.5)}"/>
-<xacro:add_leg prefix="limb3" shoulderxyz="${0.085*cos(3.*3.141592/2.5)} ${0.085*sin(3.*3.141592/2.5)} 0." shoulderrpy="0. 0. ${(3.*3.141592/2.5)}"/>
-<xacro:add_leg prefix="limb4" shoulderxyz="${0.085*cos(4.*3.141592/2.5)} ${0.085*sin(4.*3.141592/2.5)} 0." shoulderrpy="0. 0. ${(4.*3.141592/2.5)}"/>
-<xacro:add_base_plate name="upper_plate" stl_file_name="Chassi_top.stl" z="0.03"/>
-<xacro:add_base_plate name="lower_plate" stl_file_name="Chassi_bottom.stl" z="-0.03"/>
+<xacro:leg prefix="limb0" shoulderxyz="${0.085*cos(0.*3.141592/2.5)} ${0.085*sin(0.*3.141592/2.5)} 0." shoulderrpy="0. 0. ${(0.*3.141592/2.5)}"/>
+<xacro:leg prefix="limb1" shoulderxyz="${0.085*cos(1.*3.141592/2.5)} ${0.085*sin(1.*3.141592/2.5)} 0." shoulderrpy="0. 0. ${(1.*3.141592/2.5)}"/>
+<xacro:leg prefix="limb2" shoulderxyz="${0.085*cos(2.*3.141592/2.5)} ${0.085*sin(2.*3.141592/2.5)} 0." shoulderrpy="0. 0. ${(2.*3.141592/2.5)}"/>
+<xacro:leg prefix="limb3" shoulderxyz="${0.085*cos(3.*3.141592/2.5)} ${0.085*sin(3.*3.141592/2.5)} 0." shoulderrpy="0. 0. ${(3.*3.141592/2.5)}"/>
+<xacro:leg prefix="limb4" shoulderxyz="${0.085*cos(4.*3.141592/2.5)} ${0.085*sin(4.*3.141592/2.5)} 0." shoulderrpy="0. 0. ${(4.*3.141592/2.5)}"/>
 </robot>
