Commit message: add head

File: penta_description/urdf/penta.urdf.xacro (robot description, xacro)
@@ -13,5 +13,20 @@
     <parent link="base_footprint"/>
     <child link="base_link"/>
-    <origin xyz="0.0 0.0 0.05" rpy="0 0 0"/>
+    <origin xyz="0.0 0.0 0.075" rpy="0 0 0"/>
+  </joint>
+  <link name="head_link">
+    <visual>
+      <geometry>
+        <sphere radius="0.05"/>
+      </geometry>
+      <material name="green">
+        <color rgba="0 1 0 1"/>
+      </material>
+    </visual>
+  </link>
+  <joint name="head_base" type="fixed">
+    <parent link="base_link"/>
+    <child link="head_link"/>
+    <origin xyz="-0.1 0.0 0.025" rpy="0 0 0"/>
   </joint>
   <xacro:macro name="leg" params="prefix shoulderxyz shoulderrpy">

Commit message: use realrobot dimensions

File: penta_description/urdf/penta.urdf.xacro (robot description, xacro)
@@ -5,5 +5,5 @@
     <visual>
       <geometry>
-        <cylinder radius="0.10" length="0.025"/>
+        <cylinder radius="0.085" length="0.025"/>
       </geometry>
       <origin xyz="0.0 0.0 0.0" rpy="0 0 0"/>
@@ -42,7 +42,7 @@
       <visual>
         <geometry>
-          <box size="0.1 0.02 0.02"/>
+          <box size="0.0455 0.02 0.02"/>
         </geometry>
-        <origin xyz="0.05 0.0 0.0" rpy="0 0 0"/>
+        <origin xyz="0.02275 0.0 0.0" rpy="0 0 0"/>
       </visual>
     </link>
@@ -50,7 +50,7 @@
       <visual>
         <geometry>
-          <box size="0.1 0.02 0.02"/>
+          <box size="0.096 0.02 0.02"/>
         </geometry>
-        <origin xyz="0.05 0.0 0.0" rpy="0 0 0"/>
+        <origin xyz="0.048 0.0 0.0" rpy="0 0 0"/>
       </visual>
     </link>
@@ -58,7 +58,7 @@
       <visual>
         <geometry>
-          <box size="0.1 0.02 0.02"/>
+          <box size="0.158 0.02 0.02"/>
         </geometry>
-        <origin xyz="0.05 0.0 0.0" rpy="0 0 0"/>
+        <origin xyz="0.079 0.0 0.0" rpy="0 0 0"/>
       </visual>
     </link>
@@ -77,5 +77,5 @@
       <parent link="${prefix}_shoulder_link"/>
       <child link="${prefix}_upper_arm_link"/>
-      <origin xyz="0.1 0.0 0.0" rpy="-1.57 0 0"/>
+      <origin xyz="0.0455 0.0 0.0" rpy="-1.57 0 0"/>
       <axis xyz="0 0 1" />
     </joint>
@@ -83,12 +83,12 @@
       <parent link="${prefix}_upper_arm_link"/>
       <child link="${prefix}_lower_arm_link"/>
-      <origin xyz="0.1 0.0 0.0" rpy="0 0 0"/>
+      <origin xyz="0.096 0.0 0.0" rpy="0 0 0"/>
       <axis xyz="0 0 1" />
     </joint>
   </xacro:macro>
-<xacro:leg prefix="limb0" shoulderxyz="${0.1*cos(0.*3.141592/2.5)} ${0.1*sin(0.*3.141592/2.5)} 0." shoulderrpy="0. 0. ${(0.*3.141592/2.5)}"/>
-<xacro:leg prefix="limb1" shoulderxyz="${0.1*cos(1.*3.141592/2.5)} ${0.1*sin(1.*3.141592/2.5)} 0." shoulderrpy="0. 0. ${(1.*3.141592/2.5)}"/>
-<xacro:leg prefix="limb2" shoulderxyz="${0.1*cos(2.*3.141592/2.5)} ${0.1*sin(2.*3.141592/2.5)} 0." shoulderrpy="0. 0. ${(2.*3.141592/2.5)}"/>
-<xacro:leg prefix="limb3" shoulderxyz="${0.1*cos(3.*3.141592/2.5)} ${0.1*sin(3.*3.141592/2.5)} 0." shoulderrpy="0. 0. ${(3.*3.141592/2.5)}"/>
-<xacro:leg prefix="limb4" shoulderxyz="${0.1*cos(4.*3.141592/2.5)} ${0.1*sin(4.*3.141592/2.5)} 0." shoulderrpy="0. 0. ${(4.*3.141592/2.5)}"/>
+<xacro:leg prefix="limb0" shoulderxyz="${0.085*cos(0.*3.141592/2.5)} ${0.085*sin(0.*3.141592/2.5)} 0." shoulderrpy="0. 0. ${(0.*3.141592/2.5)}"/>
+<xacro:leg prefix="limb1" shoulderxyz="${0.085*cos(1.*3.141592/2.5)} ${0.085*sin(1.*3.141592/2.5)} 0." shoulderrpy="0. 0. ${(1.*3.141592/2.5)}"/>
+<xacro:leg prefix="limb2" shoulderxyz="${0.085*cos(2.*3.141592/2.5)} ${0.085*sin(2.*3.141592/2.5)} 0." shoulderrpy="0. 0. ${(2.*3.141592/2.5)}"/>
+<xacro:leg prefix="limb3" shoulderxyz="${0.085*cos(3.*3.141592/2.5)} ${0.085*sin(3.*3.141592/2.5)} 0." shoulderrpy="0. 0. ${(3.*3.141592/2.5)}"/>
+<xacro:leg prefix="limb4" shoulderxyz="${0.085*cos(4.*3.141592/2.5)} ${0.085*sin(4.*3.141592/2.5)} 0." shoulderrpy="0. 0. ${(4.*3.141592/2.5)}"/>
 </robot>

Commit message: floating base

File: penta_description/urdf/penta.urdf.xacro (robot description, xacro)
@@ -10,5 +10,5 @@
     </visual>
   </link>
-  <joint name="joint_robot_body_center" type="fixed">
+  <joint name="joint_robot_body_center" type="floating">
     <parent link="base_footprint"/>
     <child link="base_link"/>

Commit message: add 3D models

File: penta_description/urdf/penta.urdf.xacro (robot description, xacro)
@@ -1,11 +1,14 @@
 <?xml version="1.0"?>
 <robot name="penta_bot" xmlns:xacro="http://www.ros.org/wiki/xacro">
+  <xacro:property name="PI" value="3.141592" />
+  <xacro:property name="PI2" value="${PI/2}" />
+  <xacro:property name="base_visual_yaw" value="0.32" />
   <link name="base_footprint"/>
   <link name="base_link">
     <visual>
       <geometry>
-        <cylinder radius="0.085" length="0.025"/>
+        <mesh filename="package://penta_description/meshes/visual/penta_stl_v1/Chassi_middle.stl" scale="0.001 0.001 0.001"/>
       </geometry>
-      <origin xyz="0.0 0.0 0.0" rpy="0 0 0"/>
+      <origin xyz="0.0 0.0 0.0" rpy="0 0 ${base_visual_yaw}"/>
     </visual>
   </link>
@@ -18,5 +21,5 @@
     <visual>
       <geometry>
-        <sphere radius="0.05"/>
+        <sphere radius="0.01"/>
       </geometry>
       <material name="green">
@@ -30,5 +33,20 @@
     <origin xyz="-0.1 0.0 0.025" rpy="0 0 0"/>
   </joint>
-  <xacro:macro name="leg" params="prefix shoulderxyz shoulderrpy">
+  <xacro:macro name="add_base_plate" params="name stl_file_name z">
+    <link name="${name}_link">
+      <visual>
+        <geometry>
+          <mesh filename="package://penta_description/meshes/visual/penta_stl_v1/${stl_file_name}" scale="0.001 0.001 0.001"/>
+        </geometry>
+        <origin xyz="0.0 0.0 0.0" rpy="0 0 ${base_visual_yaw}"/>
+      </visual>
+    </link>
+    <joint name="${name}_joint" type="fixed">
+      <parent link="base_link"/>
+      <child link="${name}_link"/>
+    <origin xyz="0.0 0.0 ${z}" rpy="0 0 0"/>
+  </joint>
+  </xacro:macro>
+  <xacro:macro name="add_leg" params="prefix shoulderxyz shoulderrpy">
     <link name="${prefix}_shoulder_motor">
       <visual>
@@ -42,7 +60,7 @@
       <visual>
         <geometry>
-          <box size="0.0455 0.02 0.02"/>
+          <mesh filename="package://penta_description/meshes/visual/penta_stl_v1/Shoulder.stl" scale="0.001 0.001 0.001"/>
         </geometry>
-        <origin xyz="0.02275 0.0 0.0" rpy="0 0 0"/>
+        <origin xyz="0.0 0.0 0.0" rpy="-${PI2} 0 0"/>
       </visual>
     </link>
@@ -50,7 +68,7 @@
       <visual>
         <geometry>
-          <box size="0.096 0.02 0.02"/>
+          <mesh filename="package://penta_description/meshes/visual/penta_stl_v1/Upper_arm.stl" scale="0.001 0.001 0.001"/>
         </geometry>
-        <origin xyz="0.048 0.0 0.0" rpy="0 0 0"/>
+        <origin xyz="0.0 0.0 0.0" rpy="0 0 0"/>
       </visual>
     </link>
@@ -58,7 +76,7 @@
       <visual>
         <geometry>
-          <box size="0.158 0.02 0.02"/>
+          <mesh filename="package://penta_description/meshes/visual/penta_stl_v1/Lower_arm.stl" scale="0.001 0.001 0.001"/>
         </geometry>
-        <origin xyz="0.079 0.0 0.0" rpy="0 0 0"/>
+        <origin xyz="0.0 0.0 0.0" rpy="-${PI2} ${PI2} 0.4"/>
       </visual>
     </link>
@@ -87,8 +105,10 @@
     </joint>
   </xacro:macro>
-<xacro:leg prefix="limb0" shoulderxyz="${0.085*cos(0.*3.141592/2.5)} ${0.085*sin(0.*3.141592/2.5)} 0." shoulderrpy="0. 0. ${(0.*3.141592/2.5)}"/>
-<xacro:leg prefix="limb1" shoulderxyz="${0.085*cos(1.*3.141592/2.5)} ${0.085*sin(1.*3.141592/2.5)} 0." shoulderrpy="0. 0. ${(1.*3.141592/2.5)}"/>
-<xacro:leg prefix="limb2" shoulderxyz="${0.085*cos(2.*3.141592/2.5)} ${0.085*sin(2.*3.141592/2.5)} 0." shoulderrpy="0. 0. ${(2.*3.141592/2.5)}"/>
-<xacro:leg prefix="limb3" shoulderxyz="${0.085*cos(3.*3.141592/2.5)} ${0.085*sin(3.*3.141592/2.5)} 0." shoulderrpy="0. 0. ${(3.*3.141592/2.5)}"/>
-<xacro:leg prefix="limb4" shoulderxyz="${0.085*cos(4.*3.141592/2.5)} ${0.085*sin(4.*3.141592/2.5)} 0." shoulderrpy="0. 0. ${(4.*3.141592/2.5)}"/>
+<xacro:add_leg prefix="limb0" shoulderxyz="${0.085*cos(0.*3.141592/2.5)} ${0.085*sin(0.*3.141592/2.5)} 0." shoulderrpy="0. 0. ${(0.*3.141592/2.5)}"/>
+<xacro:add_leg prefix="limb1" shoulderxyz="${0.085*cos(1.*3.141592/2.5)} ${0.085*sin(1.*3.141592/2.5)} 0." shoulderrpy="0. 0. ${(1.*3.141592/2.5)}"/>
+<xacro:add_leg prefix="limb2" shoulderxyz="${0.085*cos(2.*3.141592/2.5)} ${0.085*sin(2.*3.141592/2.5)} 0." shoulderrpy="0. 0. ${(2.*3.141592/2.5)}"/>
+<xacro:add_leg prefix="limb3" shoulderxyz="${0.085*cos(3.*3.141592/2.5)} ${0.085*sin(3.*3.141592/2.5)} 0." shoulderrpy="0. 0. ${(3.*3.141592/2.5)}"/>
+<xacro:add_leg prefix="limb4" shoulderxyz="${0.085*cos(4.*3.141592/2.5)} ${0.085*sin(4.*3.141592/2.5)} 0." shoulderrpy="0. 0. ${(4.*3.141592/2.5)}"/>
+<xacro:add_base_plate name="upper_plate" stl_file_name="Chassi_top.stl" z="0.03"/>
+<xacro:add_base_plate name="lower_plate" stl_file_name="Chassi_bottom.stl" z="-0.03"/>
 </robot>

Commit message: add collision

File: penta_description/urdf/penta.urdf.xacro (robot description, xacro)
@@ -12,4 +12,10 @@
       <origin xyz="0.0 0.0 0.0" rpy="0 0 ${base_visual_yaw}"/>
     </visual>
+    <collision>
+      <geometry>
+        <mesh filename="package://penta_description/meshes/visual/penta_stl_v1/Chassi_middle.stl" scale="0.001 0.001 0.001"/>
+      </geometry>
+      <origin xyz="0.0 0.0 0.0" rpy="0 0 ${base_visual_yaw}"/>
+    </collision>
   </link>
   <joint name="joint_robot_body_center" type="floating">
@@ -80,4 +86,10 @@
         <origin xyz="0.0 0.0 0.0" rpy="-${PI2} ${PI2} 0.4"/>
       </visual>
+      <collision>
+        <geometry>
+          <mesh filename="package://penta_description/meshes/visual/penta_stl_v1/Lower_arm.stl" scale="0.001 0.001 0.001"/>
+        </geometry>
+        <origin xyz="0.0 0.0 0.0" rpy="-${PI2} ${PI2} 0.4"/>
+      </collision>
     </link>
     <joint name="${prefix}/joint_shoulder_motor" type="fixed">

Commit message: use simple collision model for the base

File: penta_description/urdf/penta.urdf.xacro (robot description, xacro)
@@ -14,7 +14,7 @@
     <collision>
       <geometry>
-        <mesh filename="package://penta_description/meshes/visual/penta_stl_v1/Chassi_middle.stl" scale="0.001 0.001 0.001"/>
+        <cylinder radius="0.15" length="0.085"/>
       </geometry>
-      <origin xyz="0.0 0.0 0.0" rpy="0 0 ${base_visual_yaw}"/>
+      <origin xyz="0.0 0.0 0.0" rpy="0 0 0"/>
     </collision>
   </link>

Commit message: wip gazebo

File: penta_description/urdf/penta.urdf.xacro (robot description, xacro)
@@ -18,4 +18,9 @@
       <origin xyz="0.0 0.0 0.0" rpy="0 0 0"/>
     </collision>
+    <inertial>
+      <origin rpy="0 0 0" xyz="0.0 0.0 0.0"/>
+      <mass value="1.0"/>
+      <inertia ixx="1.0" ixy="0" ixz="0" iyy="1.0" iyz="0" izz="1.0"/>
+    </inertial>
   </link>
   <joint name="joint_robot_body_center" type="floating">
@@ -62,4 +67,9 @@
         <origin xyz="0.0 0.0 0.0" rpy="0 0 0"/>
       </visual>
+      <inertial>
+        <origin rpy="0 0 0" xyz="0.0 0.0 0.0"/>
+        <mass value="1.0"/>
+        <inertia ixx="1.0" ixy="0" ixz="0" iyy="1.0" iyz="0" izz="1.0"/>
+      </inertial>
     </link>
     <link name="${prefix}_shoulder_link">
@@ -70,4 +80,9 @@
         <origin xyz="0.0 0.0 0.0" rpy="-${PI2} 0 0"/>
       </visual>
+      <inertial>
+        <origin rpy="0 0 0" xyz="0.0 0.0 0.0"/>
+        <mass value="1.0"/>
+        <inertia ixx="1.0" ixy="0" ixz="0" iyy="1.0" iyz="0" izz="1.0"/>
+      </inertial>
     </link>
     <link name="${prefix}_upper_arm_link">
@@ -78,4 +93,9 @@
         <origin xyz="0.0 0.0 0.0" rpy="0 0 0"/>
       </visual>
+      <inertial>
+        <origin rpy="0 0 0" xyz="0.0 0.0 0.0"/>
+        <mass value="1.0"/>
+        <inertia ixx="1.0" ixy="0" ixz="0" iyy="1.0" iyz="0" izz="1.0"/>
+      </inertial>
     </link>
     <link name="${prefix}_lower_arm_link">
@@ -92,4 +112,9 @@
         <origin xyz="0.0 0.0 0.0" rpy="-${PI2} ${PI2} 0.4"/>
       </collision>
+      <inertial>
+        <origin rpy="0 0 0" xyz="0.0 0.0 0.0"/>
+        <mass value="1.0"/>
+        <inertia ixx="1.0" ixy="0" ixz="0" iyy="1.0" iyz="0" izz="1.0"/>
+      </inertial>
     </link>
     <joint name="${prefix}/joint_shoulder_motor" type="fixed">

Commit message: wip

File: penta_description/urdf/penta.urdf.xacro (robot description, xacro)
@@ -4,4 +4,14 @@
   <xacro:property name="PI2" value="${PI/2}" />
   <xacro:property name="base_visual_yaw" value="0.32" />
+  <xacro:macro name="add_material_green">
+      <material name="green">
+        <color rgba="0 1 0 1"/>
+      </material>
+  </xacro:macro>
+  <xacro:macro name="add_material_red">
+      <material name="red">
+        <color rgba="1 0 0 1"/>
+      </material>
+  </xacro:macro>
   <link name="base_footprint"/>
   <link name="base_link">
@@ -11,4 +21,5 @@
       </geometry>
       <origin xyz="0.0 0.0 0.0" rpy="0 0 ${base_visual_yaw}"/>
+      <xacro:add_material_red/>
     </visual>
     <collision>
@@ -24,5 +35,5 @@
     </inertial>
   </link>
-  <joint name="joint_robot_body_center" type="floating">
+  <joint name="joint_robot_body_center" type="fixed">
     <parent link="base_footprint"/>
     <child link="base_link"/>
@@ -34,7 +45,5 @@
         <sphere radius="0.01"/>
       </geometry>
-      <material name="green">
-        <color rgba="0 1 0 1"/>
-      </material>
+      <xacro:add_material_green/>
     </visual>
   </link>
@@ -51,4 +60,5 @@
         </geometry>
         <origin xyz="0.0 0.0 0.0" rpy="0 0 ${base_visual_yaw}"/>
+        <xacro:add_material_red/>
       </visual>
     </link>
@@ -66,4 +76,5 @@
         </geometry>
         <origin xyz="0.0 0.0 0.0" rpy="0 0 0"/>
+        <xacro:add_material_red/>
       </visual>
       <inertial>
@@ -79,4 +90,5 @@
         </geometry>
         <origin xyz="0.0 0.0 0.0" rpy="-${PI2} 0 0"/>
+        <xacro:add_material_red/>
       </visual>
       <inertial>
@@ -92,4 +104,5 @@
         </geometry>
         <origin xyz="0.0 0.0 0.0" rpy="0 0 0"/>
+        <xacro:add_material_red/>
       </visual>
       <inertial>
@@ -105,4 +118,5 @@
         </geometry>
         <origin xyz="0.0 0.0 0.0" rpy="-${PI2} ${PI2} 0.4"/>
+        <xacro:add_material_red/>
       </visual>
       <collision>

Commit message: move limb macro into separate file

File: penta_description/urdf/penta.urdf.xacro (robot description, xacro)
@@ -4,4 +4,5 @@
   <xacro:property name="PI2" value="${PI/2}" />
   <xacro:property name="base_visual_yaw" value="0.32" />
+  <xacro:include filename="$(find penta_description)/urdf/single_limb.urdf.xacro" />
   <xacro:macro name="add_material_green">
       <material name="green">
@@ -69,91 +70,4 @@
   </joint>
   </xacro:macro>
-  <xacro:macro name="add_leg" params="prefix shoulderxyz shoulderrpy">
-    <link name="${prefix}_shoulder_motor">
-      <visual>
-        <geometry>
-          <cylinder radius="0.0350" length="0.035"/>
-        </geometry>
-        <origin xyz="0.0 0.0 0.0" rpy="0 0 0"/>
-        <xacro:add_material_red/>
-      </visual>
-      <inertial>
-        <origin rpy="0 0 0" xyz="0.0 0.0 0.0"/>
-        <mass value="1.0"/>
-        <inertia ixx="1.0" ixy="0" ixz="0" iyy="1.0" iyz="0" izz="1.0"/>
-      </inertial>
-    </link>
-    <link name="${prefix}_shoulder_link">
-      <visual>
-        <geometry>
-          <mesh filename="package://penta_description/meshes/visual/penta_stl_v1/Shoulder.stl" scale="0.001 0.001 0.001"/>
-        </geometry>
-        <origin xyz="0.0 0.0 0.0" rpy="-${PI2} 0 0"/>
-        <xacro:add_material_red/>
-      </visual>
-      <inertial>
-        <origin rpy="0 0 0" xyz="0.0 0.0 0.0"/>
-        <mass value="1.0"/>
-        <inertia ixx="1.0" ixy="0" ixz="0" iyy="1.0" iyz="0" izz="1.0"/>
-      </inertial>
-    </link>
-    <link name="${prefix}_upper_arm_link">
-      <visual>
-        <geometry>
-          <mesh filename="package://penta_description/meshes/visual/penta_stl_v1/Upper_arm.stl" scale="0.001 0.001 0.001"/>
-        </geometry>
-        <origin xyz="0.0 0.0 0.0" rpy="0 0 0"/>
-        <xacro:add_material_red/>
-      </visual>
-      <inertial>
-        <origin rpy="0 0 0" xyz="0.0 0.0 0.0"/>
-        <mass value="1.0"/>
-        <inertia ixx="1.0" ixy="0" ixz="0" iyy="1.0" iyz="0" izz="1.0"/>
-      </inertial>
-    </link>
-    <link name="${prefix}_lower_arm_link">
-      <visual>
-        <geometry>
-          <mesh filename="package://penta_description/meshes/visual/penta_stl_v1/Lower_arm.stl" scale="0.001 0.001 0.001"/>
-        </geometry>
-        <origin xyz="0.0 0.0 0.0" rpy="-${PI2} ${PI2} 0.4"/>
-        <xacro:add_material_red/>
-      </visual>
-      <collision>
-        <geometry>
-          <mesh filename="package://penta_description/meshes/visual/penta_stl_v1/Lower_arm.stl" scale="0.001 0.001 0.001"/>
-        </geometry>
-        <origin xyz="0.0 0.0 0.0" rpy="-${PI2} ${PI2} 0.4"/>
-      </collision>
-      <inertial>
-        <origin rpy="0 0 0" xyz="0.0 0.0 0.0"/>
-        <mass value="1.0"/>
-        <inertia ixx="1.0" ixy="0" ixz="0" iyy="1.0" iyz="0" izz="1.0"/>
-      </inertial>
-    </link>
-    <joint name="${prefix}/joint_shoulder_motor" type="fixed">
-      <parent link="base_link"/>
-      <child link="${prefix}_shoulder_motor"/>
-      <origin xyz="${shoulderxyz}" rpy="${shoulderrpy}"/>
-    </joint>
-    <joint name="${prefix}/joint0" type="continuous">
-      <parent link="${prefix}_shoulder_motor"/>
-      <child link="${prefix}_shoulder_link"/>
-      <origin xyz="0.0 0.0 0.0" rpy="0 0 0"/>
-      <axis xyz="0 0 1" />
-    </joint>
-    <joint name="${prefix}/joint1" type="continuous">
-      <parent link="${prefix}_shoulder_link"/>
-      <child link="${prefix}_upper_arm_link"/>
-      <origin xyz="0.0455 0.0 0.0" rpy="-1.57 0 0"/>
-      <axis xyz="0 0 1" />
-    </joint>
-    <joint name="${prefix}/joint2" type="continuous">
-      <parent link="${prefix}_upper_arm_link"/>
-      <child link="${prefix}_lower_arm_link"/>
-      <origin xyz="0.096 0.0 0.0" rpy="0 0 0"/>
-      <axis xyz="0 0 1" />
-    </joint>
-  </xacro:macro>
 <xacro:add_leg prefix="limb0" shoulderxyz="${0.085*cos(0.*3.141592/2.5)} ${0.085*sin(0.*3.141592/2.5)} 0." shoulderrpy="0. 0. ${(0.*3.141592/2.5)}"/>
 <xacro:add_leg prefix="limb1" shoulderxyz="${0.085*cos(1.*3.141592/2.5)} ${0.085*sin(1.*3.141592/2.5)} 0." shoulderrpy="0. 0. ${(1.*3.141592/2.5)}"/>

File: penta_description/urdf/single_limb.urdf.xacro (robot description, xacro)
@@ -1,19 +1,5 @@
 <?xml version="1.0"?>
-<robot name="penta_bot" xmlns:xacro="http://www.ros.org/wiki/xacro">
-  <link name="base_footprint"/>
-  <link name="base_link">
-    <visual>
-      <geometry>
-        <cylinder radius="0.10" length="0.025"/>
-      </geometry>
-      <origin xyz="0.0 0.0 0.0" rpy="0 0 0"/>
-    </visual>
-  </link>
-  <joint name="joint_robot_body_center" type="fixed">
-    <parent link="base_footprint"/>
-    <child link="base_link"/>
-    <origin xyz="0.0 0.0 0.05" rpy="0 0 0"/>
-  </joint>
-  <xacro:macro name="leg" params="prefix">
+<robot xmlns:xacro="http://www.ros.org/wiki/xacro">
+  <xacro:macro name="add_leg" params="prefix shoulderxyz shoulderrpy">
     <link name="${prefix}_shoulder_motor">
       <visual>
@@ -22,36 +8,66 @@
         </geometry>
         <origin xyz="0.0 0.0 0.0" rpy="0 0 0"/>
+        <xacro:add_material_red/>
       </visual>
+      <inertial>
+        <origin rpy="0 0 0" xyz="0.0 0.0 0.0"/>
+        <mass value="1.0"/>
+        <inertia ixx="1.0" ixy="0" ixz="0" iyy="1.0" iyz="0" izz="1.0"/>
+      </inertial>
     </link>
     <link name="${prefix}_shoulder_link">
       <visual>
         <geometry>
-          <box size="0.1 0.02 0.02"/>
+          <mesh filename="package://penta_description/meshes/visual/penta_stl_v1/Shoulder.stl" scale="0.001 0.001 0.001"/>
         </geometry>
-        <origin xyz="0.05 0.0 0.0" rpy="0 0 0"/>
+        <origin xyz="0.0 0.0 0.0" rpy="-${PI2} 0 0"/>
+        <xacro:add_material_red/>
       </visual>
+      <inertial>
+        <origin rpy="0 0 0" xyz="0.0 0.0 0.0"/>
+        <mass value="1.0"/>
+        <inertia ixx="1.0" ixy="0" ixz="0" iyy="1.0" iyz="0" izz="1.0"/>
+      </inertial>
     </link>
     <link name="${prefix}_upper_arm_link">
       <visual>
         <geometry>
-          <box size="0.1 0.02 0.02"/>
+          <mesh filename="package://penta_description/meshes/visual/penta_stl_v1/Upper_arm.stl" scale="0.001 0.001 0.001"/>
         </geometry>
-        <origin xyz="0.05 0.0 0.0" rpy="0 0 0"/>
+        <origin xyz="0.0 0.0 0.0" rpy="0 0 0"/>
+        <xacro:add_material_red/>
       </visual>
+      <inertial>
+        <origin rpy="0 0 0" xyz="0.0 0.0 0.0"/>
+        <mass value="1.0"/>
+        <inertia ixx="1.0" ixy="0" ixz="0" iyy="1.0" iyz="0" izz="1.0"/>
+      </inertial>
     </link>
     <link name="${prefix}_lower_arm_link">
       <visual>
         <geometry>
-          <box size="0.1 0.02 0.02"/>
+          <mesh filename="package://penta_description/meshes/visual/penta_stl_v1/Lower_arm.stl" scale="0.001 0.001 0.001"/>
         </geometry>
-        <origin xyz="0.05 0.0 0.0" rpy="0 0 0"/>
+        <origin xyz="0.0 0.0 0.0" rpy="-${PI2} ${PI2} 0.4"/>
+        <xacro:add_material_red/>
       </visual>
+      <collision>
+        <geometry>
+          <mesh filename="package://penta_description/meshes/visual/penta_stl_v1/Lower_arm.stl" scale="0.001 0.001 0.001"/>
+        </geometry>
+        <origin xyz="0.0 0.0 0.0" rpy="-${PI2} ${PI2} 0.4"/>
+      </collision>
+      <inertial>
+        <origin rpy="0 0 0" xyz="0.0 0.0 0.0"/>
+        <mass value="1.0"/>
+        <inertia ixx="1.0" ixy="0" ixz="0" iyy="1.0" iyz="0" izz="1.0"/>
+      </inertial>
     </link>
-    <joint name="${prefix}_joint_shoulder_motor" type="fixed">
+    <joint name="${prefix}/joint_shoulder_motor" type="fixed">
       <parent link="base_link"/>
       <child link="${prefix}_shoulder_motor"/>
-      <origin xyz="0.1 0.0 0.0" rpy="0 0 0"/>
+      <origin xyz="${shoulderxyz}" rpy="${shoulderrpy}"/>
     </joint>
-    <joint name="${prefix}_joint0" type="continuous">
+    <joint name="${prefix}/joint0" type="continuous">
       <parent link="${prefix}_shoulder_motor"/>
       <child link="${prefix}_shoulder_link"/>
@@ -59,17 +75,16 @@
       <axis xyz="0 0 1" />
     </joint>
-    <joint name="${prefix}_joint1" type="continuous">
+    <joint name="${prefix}/joint1" type="continuous">
       <parent link="${prefix}_shoulder_link"/>
       <child link="${prefix}_upper_arm_link"/>
-      <origin xyz="0.1 0.0 0.0" rpy="-1.57 0 0"/>
+      <origin xyz="0.0455 0.0 0.0" rpy="-1.57 0 0"/>
       <axis xyz="0 0 1" />
     </joint>
-    <joint name="${prefix}_joint2" type="continuous">
+    <joint name="${prefix}/joint2" type="continuous">
       <parent link="${prefix}_upper_arm_link"/>
       <child link="${prefix}_lower_arm_link"/>
-      <origin xyz="0.1 0.0 0.0" rpy="0 0 0"/>
+      <origin xyz="0.096 0.0 0.0" rpy="0 0 0"/>
       <axis xyz="0 0 1" />
     </joint>
   </xacro:macro>
-  <xacro:leg prefix="limb0" />
 </robot>
