Commit message: gazebo sim

File: penta_description/urdf/penta.urdf.xacro (robot description, xacro)
@@ -77,3 +77,8 @@
 <xacro:add_base_plate name="upper_plate" stl_file_name="Chassi_top.stl" z="0.03"/>
 <xacro:add_base_plate name="lower_plate" stl_file_name="Chassi_bottom.stl" z="-0.03"/>
+<gazebo>
+  <plugin filename="libgazebo_ros2_control.so" name="gazebo_ros2_control" >
+    <parameters>$(find penta_description)/config/ros2_control_params.yaml</parameters>
+  </plugin>
+</gazebo>
 </robot>

File: penta_description/urdf/single_limb.urdf.xacro (robot description, xacro)
@@ -87,4 +87,56 @@
       <axis xyz="0 0 1" />
     </joint>
+    <!-- ros2_control interfaces for each joint -->
+    <ros2_control name="${prefix}_ros2_control" type="system">
+      <hardware>
+        <plugin>gazebo_ros2_control/GazeboSystem</plugin>
+      </hardware>
+      <joint name="${prefix}/joint0">
+        <command_interface name="position"/>
+        <state_interface name="position"/>
+        <state_interface name="velocity"/>
+      </joint>
+      <joint name="${prefix}/joint1">
+        <command_interface name="position"/>
+        <state_interface name="position"/>
+        <state_interface name="velocity"/>
+      </joint>
+      <joint name="${prefix}/joint2">
+        <command_interface name="position"/>
+        <state_interface name="position"/>
+        <state_interface name="velocity"/>
+      </joint>
+    </ros2_control>
+    <!-- Transmission blocks -->
+    <transmission name="${prefix}_joint0_trans">
+      <type>transmission_interface/SimpleTransmission</type>
+      <joint name="${prefix}/joint0">
+        <hardwareInterface>hardware_interface/PositionJointInterface</hardwareInterface>
+      </joint>
+      <actuator name="${prefix}_motor0">
+        <hardwareInterface>hardware_interface/PositionJointInterface</hardwareInterface>
+        <mechanicalReduction>1</mechanicalReduction>
+      </actuator>
+    </transmission>
+    <transmission name="${prefix}_joint1_trans">
+      <type>transmission_interface/SimpleTransmission</type>
+      <joint name="${prefix}/joint1">
+        <hardwareInterface>hardware_interface/PositionJointInterface</hardwareInterface>
+      </joint>
+      <actuator name="${prefix}_motor1">
+        <hardwareInterface>hardware_interface/PositionJointInterface</hardwareInterface>
+        <mechanicalReduction>1</mechanicalReduction>
+      </actuator>
+    </transmission>
+    <transmission name="${prefix}_joint2_trans">
+      <type>transmission_interface/SimpleTransmission</type>
+      <joint name="${prefix}/joint2">
+        <hardwareInterface>hardware_interface/PositionJointInterface</hardwareInterface>
+      </joint>
+      <actuator name="${prefix}_motor2">
+        <hardwareInterface>hardware_interface/PositionJointInterface</hardwareInterface>
+        <mechanicalReduction>1</mechanicalReduction>
+      </actuator>
+    </transmission>
   </xacro:macro>
 </robot>

Commit message: the robot as xacro

File: penta_description/urdf/penta.urdf.xacro (robot description, xacro)
@@ -1,84 +1,14 @@
 <?xml version="1.0"?>
 <robot name="penta_bot" xmlns:xacro="http://www.ros.org/wiki/xacro">
-  <xacro:property name="PI" value="3.141592" />
-  <xacro:property name="PI2" value="${PI/2}" />
-  <xacro:property name="base_visual_yaw" value="0.32" />
-  <xacro:include filename="$(find penta_description)/urdf/single_limb.urdf.xacro" />
-  <xacro:macro name="add_material_green">
-      <material name="green">
-        <color rgba="0 1 0 1"/>
-      </material>
-  </xacro:macro>
-  <xacro:macro name="add_material_red">
-      <material name="red">
-        <color rgba="1 0 0 1"/>
-      </material>
-  </xacro:macro>
-  <link name="base_footprint"/>
-  <link name="base_link">
-    <visual>
-      <geometry>
-        <mesh filename="package://penta_description/meshes/visual/penta_stl_v1/Chassi_middle.stl" scale="0.001 0.001 0.001"/>
-      </geometry>
-      <origin xyz="0.0 0.0 0.0" rpy="0 0 ${base_visual_yaw}"/>
-      <xacro:add_material_red/>
-    </visual>
-    <collision>
-      <geometry>
-        <cylinder radius="0.15" length="0.085"/>
-      </geometry>
-      <origin xyz="0.0 0.0 0.0" rpy="0 0 0"/>
-    </collision>
-    <inertial>
-      <origin rpy="0 0 0" xyz="0.0 0.0 0.0"/>
-      <mass value="1.0"/>
-      <inertia ixx="1.0" ixy="0" ixz="0" iyy="1.0" iyz="0" izz="1.0"/>
-    </inertial>
-  </link>
-  <joint name="joint_robot_body_center" type="fixed">
-    <parent link="base_footprint"/>
-    <child link="base_link"/>
-    <origin xyz="0.0 0.0 0.075" rpy="0 0 0"/>
-  </joint>
-  <link name="head_link">
-    <visual>
-      <geometry>
-        <sphere radius="0.01"/>
-      </geometry>
-      <xacro:add_material_green/>
-    </visual>
-  </link>
-  <joint name="head_base" type="fixed">
-    <parent link="base_link"/>
-    <child link="head_link"/>
-    <origin xyz="-0.1 0.0 0.025" rpy="0 0 0"/>
-  </joint>
-  <xacro:macro name="add_base_plate" params="name stl_file_name z">
-    <link name="${name}_link">
-      <visual>
-        <geometry>
-          <mesh filename="package://penta_description/meshes/visual/penta_stl_v1/${stl_file_name}" scale="0.001 0.001 0.001"/>
-        </geometry>
-        <origin xyz="0.0 0.0 0.0" rpy="0 0 ${base_visual_yaw}"/>
-        <xacro:add_material_red/>
-      </visual>
-    </link>
-    <joint name="${name}_joint" type="fixed">
-      <parent link="base_link"/>
-      <child link="${name}_link"/>
-    <origin xyz="0.0 0.0 ${z}" rpy="0 0 0"/>
-  </joint>
-  </xacro:macro>
-<xacro:add_leg prefix="limb0" shoulderxyz="${0.085*cos(0.*3.141592/2.5)} ${0.085*sin(0.*3.141592/2.5)} 0." shoulderrpy="0. 0. ${(0.*3.141592/2.5)}"/>
-<xacro:add_leg prefix="limb1" shoulderxyz="${0.085*cos(1.*3.141592/2.5)} ${0.085*sin(1.*3.141592/2.5)} 0." shoulderrpy="0. 0. ${(1.*3.141592/2.5)}"/>
-<xacro:add_leg prefix="limb2" shoulderxyz="${0.085*cos(2.*3.141592/2.5)} ${0.085*sin(2.*3.141592/2.5)} 0." shoulderrpy="0. 0. ${(2.*3.141592/2.5)}"/>
-<xacro:add_leg prefix="limb3" shoulderxyz="${0.085*cos(3.*3.141592/2.5)} ${0.085*sin(3.*3.141592/2.5)} 0." shoulderrpy="0. 0. ${(3.*3.141592/2.5)}"/>
-<xacro:add_leg prefix="limb4" shoulderxyz="${0.085*cos(4.*3.141592/2.5)} ${0.085*sin(4.*3.141592/2.5)} 0." shoulderrpy="0. 0. ${(4.*3.141592/2.5)}"/>
-<xacro:add_base_plate name="upper_plate" stl_file_name="Chassi_top.stl" z="0.03"/>
-<xacro:add_base_plate name="lower_plate" stl_file_name="Chassi_bottom.stl" z="-0.03"/>
-<gazebo>
-  <plugin filename="libgazebo_ros2_control.so" name="gazebo_ros2_control" >
-    <parameters>$(find penta_description)/config/ros2_control_params.yaml</parameters>
-  </plugin>
-</gazebo>
+  <xacro:include filename="$(find penta_description)/urdf/penta_robot_macro.urdf.xacro" />
+  <xacro:add_penta_bot/>
+  <!-- gazebo ros2_control plugins -->
+  <gazebo>
+      <plugin filename="gz-sim-joint-state-publisher-system" name="gz::sim::systems::JointStatePublisher">
+          <topic>joint_states</topic>
+      </plugin>
+      <plugin filename="gz_ros2_control-system" name="gz_ros2_control::GazeboSimROS2ControlPlugin">
+          <parameters>$(find penta_description)/config/ros2_control_params.yaml</parameters>
+      </plugin>
+  </gazebo>
 </robot>

Commit message: experminting with dynamixel

File: penta_description/urdf/penta.urdf.xacro (robot description, xacro)
@@ -1,4 +1,10 @@
 <?xml version="1.0"?>
 <robot name="penta_bot" xmlns:xacro="http://www.ros.org/wiki/xacro">
+  <xacro:arg name="prefix" default="" />
+  <xacro:arg name="enable_gazebo" default="true" />
+  <xacro:arg name="use_real_dynamixel_motor" default="false" />
+  <xacro:arg name="use_fake_hardware" default="false" />
+  <xacro:arg name="fake_sensor_commands" default="false" />
+  <xacro:arg name="port_name" default="/dev/ttyUSB0" />
   <xacro:property name="PI" value="3.141592" />
   <xacro:property name="PI2" value="${PI/2}" />
@@ -70,15 +76,30 @@
   </joint>
   </xacro:macro>
-<xacro:add_leg prefix="limb0" shoulderxyz="${0.085*cos(0.*3.141592/2.5)} ${0.085*sin(0.*3.141592/2.5)} 0." shoulderrpy="0. 0. ${(0.*3.141592/2.5)}"/>
-<xacro:add_leg prefix="limb1" shoulderxyz="${0.085*cos(1.*3.141592/2.5)} ${0.085*sin(1.*3.141592/2.5)} 0." shoulderrpy="0. 0. ${(1.*3.141592/2.5)}"/>
-<xacro:add_leg prefix="limb2" shoulderxyz="${0.085*cos(2.*3.141592/2.5)} ${0.085*sin(2.*3.141592/2.5)} 0." shoulderrpy="0. 0. ${(2.*3.141592/2.5)}"/>
-<xacro:add_leg prefix="limb3" shoulderxyz="${0.085*cos(3.*3.141592/2.5)} ${0.085*sin(3.*3.141592/2.5)} 0." shoulderrpy="0. 0. ${(3.*3.141592/2.5)}"/>
-<xacro:add_leg prefix="limb4" shoulderxyz="${0.085*cos(4.*3.141592/2.5)} ${0.085*sin(4.*3.141592/2.5)} 0." shoulderrpy="0. 0. ${(4.*3.141592/2.5)}"/>
+<xacro:add_leg prefix="limb0" shoulderxyz="${0.085*cos(0.*3.141592/2.5)} ${0.085*sin(0.*3.141592/2.5)} 0." shoulderrpy="0. 0. ${(0.*3.141592/2.5)}" enable_gazebo="$(arg enable_gazebo)"/>
+<xacro:add_leg prefix="limb1" shoulderxyz="${0.085*cos(1.*3.141592/2.5)} ${0.085*sin(1.*3.141592/2.5)} 0." shoulderrpy="0. 0. ${(1.*3.141592/2.5)}" enable_gazebo="$(arg enable_gazebo)"/>
+<xacro:add_leg prefix="limb2" shoulderxyz="${0.085*cos(2.*3.141592/2.5)} ${0.085*sin(2.*3.141592/2.5)} 0." shoulderrpy="0. 0. ${(2.*3.141592/2.5)}" enable_gazebo="$(arg enable_gazebo)"/>
+<xacro:add_leg prefix="limb3" shoulderxyz="${0.085*cos(3.*3.141592/2.5)} ${0.085*sin(3.*3.141592/2.5)} 0." shoulderrpy="0. 0. ${(3.*3.141592/2.5)}" enable_gazebo="$(arg enable_gazebo)"/>
+<xacro:add_leg prefix="limb4" shoulderxyz="${0.085*cos(4.*3.141592/2.5)} ${0.085*sin(4.*3.141592/2.5)} 0." shoulderrpy="0. 0. ${(4.*3.141592/2.5)}" enable_gazebo="$(arg enable_gazebo)"/>
 <xacro:add_base_plate name="upper_plate" stl_file_name="Chassi_top.stl" z="0.03"/>
 <xacro:add_base_plate name="lower_plate" stl_file_name="Chassi_bottom.stl" z="-0.03"/>
-<gazebo>
-  <plugin filename="libgazebo_ros2_control.so" name="gazebo_ros2_control" >
-    <parameters>$(find penta_description)/config/ros2_control_params.yaml</parameters>
-  </plugin>
-</gazebo>
+<xacro:if value="$(arg enable_gazebo)">
+  <gazebo>
+    <plugin filename="libgazebo_ros2_control.so" name="gazebo_ros2_control" >
+      <parameters>$(find penta_description)/config/ros2_control_params.yaml</parameters>
+    </plugin>
+  </gazebo>
+</xacro:if>
+<xacro:unless value="$(arg enable_gazebo)">
+  <xacro:if value="$(arg use_real_dynamixel_motor)">
+    <xacro:include filename="$(find penta_description)/ros2_control/penta_dynamixel_system.ros2_control.xacro" />
+    <xacro:add_penta_dynamixel_control_system
+      name="PentaDynamixelControlSystem"
+      prefix="$(arg prefix)"
+      enable_gazebo="$(arg enable_gazebo)"
+      use_real_dynamixel_motor="$(arg use_real_dynamixel_motor)"
+      use_fake_hardware="$(arg use_fake_hardware)"
+      fake_sensor_commands="$(arg fake_sensor_commands)"
+      port_name="$(arg port_name)"/>
+  </xacro:if>
+</xacro:unless>
 </robot>

File: penta_description/urdf/single_limb.urdf.xacro (robot description, xacro)
@@ -1,5 +1,5 @@
 <?xml version="1.0"?>
 <robot xmlns:xacro="http://www.ros.org/wiki/xacro">
-  <xacro:macro name="add_leg" params="prefix shoulderxyz shoulderrpy">
+  <xacro:macro name="add_leg" params="prefix shoulderxyz shoulderrpy enable_gazebo:=false">
     <link name="${prefix}_shoulder_motor">
       <visual>
@@ -133,4 +133,5 @@
       <origin xyz="0.0 0.0 0.0" rpy="0 0 0"/>
     </joint>
+  <xacro:if value="$(arg enable_gazebo)">
     <!-- ros2_control interfaces for each joint -->
     <ros2_control name="${prefix}_ros2_control" type="system">
@@ -185,4 +186,5 @@
       </actuator>
     </transmission>
+  </xacro:if>
   </xacro:macro>
 </robot>

Commit message: fix rviz not finding stl files

File: penta_description/urdf/penta.urdf.xacro (robot description, xacro)
@@ -19,5 +19,5 @@
     <visual>
       <geometry>
-        <mesh filename="package://penta_description/meshes/visual/penta_stl_v1/Chassi_middle.stl" scale="0.001 0.001 0.001"/>
+        <mesh filename="file://$(find penta_description)/meshes/visual/penta_stl_v1/Chassi_middle.stl" scale="0.001 0.001 0.001"/>
       </geometry>
       <origin xyz="0.0 0.0 0.0" rpy="0 0 ${base_visual_yaw}"/>
@@ -58,5 +58,5 @@
       <visual>
         <geometry>
-          <mesh filename="package://penta_description/meshes/visual/penta_stl_v1/${stl_file_name}" scale="0.001 0.001 0.001"/>
+          <mesh filename="file://$(find penta_description)/meshes/visual/penta_stl_v1/${stl_file_name}" scale="0.001 0.001 0.001"/>
         </geometry>
         <origin xyz="0.0 0.0 0.0" rpy="0 0 ${base_visual_yaw}"/>

File: penta_description/urdf/single_limb.urdf.xacro (robot description, xacro)
@@ -19,5 +19,5 @@
       <visual>
         <geometry>
-          <mesh filename="package://penta_description/meshes/visual/penta_stl_v1/Shoulder.stl" scale="0.001 0.001 0.001"/>
+          <mesh filename="file://$(find penta_description)/meshes/visual/penta_stl_v1/Shoulder.stl" scale="0.001 0.001 0.001"/>
         </geometry>
         <origin xyz="0.0 0.0 0.0" rpy="-${PI2} 0 0"/>
@@ -33,5 +33,5 @@
       <visual>
         <geometry>
-          <mesh filename="package://penta_description/meshes/visual/penta_stl_v1/Upper_arm.stl" scale="0.001 0.001 0.001"/>
+          <mesh filename="file://$(find penta_description)/meshes/visual/penta_stl_v1/Upper_arm.stl" scale="0.001 0.001 0.001"/>
         </geometry>
         <origin xyz="0.0 0.0 0.0" rpy="0 0 0"/>
@@ -47,5 +47,5 @@
       <visual>
         <geometry>
-          <mesh filename="package://penta_description/meshes/visual/penta_stl_v1/Lower_arm.stl" scale="0.001 0.001 0.001"/>
+          <mesh filename="file://$(find penta_description)/meshes/visual/penta_stl_v1/Lower_arm.stl" scale="0.001 0.001 0.001"/>
         </geometry>
         <origin xyz="0.0 0.0 0.0" rpy="-${PI2} ${PI2} 0.41"/>

Commit message: use xacro args to enable/activate gazebo_ros2_control or pca9685 ros2 control

File: penta_description/urdf/penta.urdf.xacro (robot description, xacro)
@@ -1,4 +1,6 @@
 <?xml version="1.0"?>
 <robot name="penta_bot" xmlns:xacro="http://www.ros.org/wiki/xacro">
+  <xacro:arg name="use_gazebo_simulation" default="False" />
+  <xacro:arg name="use_pca9685_ros2_control" default="False" />
   <xacro:property name="PI" value="3.141592" />
   <xacro:property name="PI2" value="${PI/2}" />
@@ -70,18 +72,22 @@
   </joint>
   </xacro:macro>
-<xacro:add_leg prefix="limb0" shoulderxyz="${0.085*cos(0.*3.141592/2.5)} ${0.085*sin(0.*3.141592/2.5)} 0." shoulderrpy="0. 0. ${(0.*3.141592/2.5)}"/>
-<xacro:add_leg prefix="limb1" shoulderxyz="${0.085*cos(1.*3.141592/2.5)} ${0.085*sin(1.*3.141592/2.5)} 0." shoulderrpy="0. 0. ${(1.*3.141592/2.5)}"/>
-<xacro:add_leg prefix="limb2" shoulderxyz="${0.085*cos(2.*3.141592/2.5)} ${0.085*sin(2.*3.141592/2.5)} 0." shoulderrpy="0. 0. ${(2.*3.141592/2.5)}"/>
-<xacro:add_leg prefix="limb3" shoulderxyz="${0.085*cos(3.*3.141592/2.5)} ${0.085*sin(3.*3.141592/2.5)} 0." shoulderrpy="0. 0. ${(3.*3.141592/2.5)}"/>
-<xacro:add_leg prefix="limb4" shoulderxyz="${0.085*cos(4.*3.141592/2.5)} ${0.085*sin(4.*3.141592/2.5)} 0." shoulderrpy="0. 0. ${(4.*3.141592/2.5)}"/>
+<xacro:add_leg prefix="limb0" shoulderxyz="${0.085*cos(0.*3.141592/2.5)} ${0.085*sin(0.*3.141592/2.5)} 0." shoulderrpy="0. 0. ${(0.*3.141592/2.5)}" use_gazebo_simulation="$(arg use_gazebo_simulation)"/>
+<xacro:add_leg prefix="limb1" shoulderxyz="${0.085*cos(1.*3.141592/2.5)} ${0.085*sin(1.*3.141592/2.5)} 0." shoulderrpy="0. 0. ${(1.*3.141592/2.5)}" use_gazebo_simulation="$(arg use_gazebo_simulation)"/>
+<xacro:add_leg prefix="limb2" shoulderxyz="${0.085*cos(2.*3.141592/2.5)} ${0.085*sin(2.*3.141592/2.5)} 0." shoulderrpy="0. 0. ${(2.*3.141592/2.5)}" use_gazebo_simulation="$(arg use_gazebo_simulation)"/>
+<xacro:add_leg prefix="limb3" shoulderxyz="${0.085*cos(3.*3.141592/2.5)} ${0.085*sin(3.*3.141592/2.5)} 0." shoulderrpy="0. 0. ${(3.*3.141592/2.5)}" use_gazebo_simulation="$(arg use_gazebo_simulation)"/>
+<xacro:add_leg prefix="limb4" shoulderxyz="${0.085*cos(4.*3.141592/2.5)} ${0.085*sin(4.*3.141592/2.5)} 0." shoulderrpy="0. 0. ${(4.*3.141592/2.5)}" use_gazebo_simulation="$(arg use_gazebo_simulation)"/>
 <xacro:add_base_plate name="upper_plate" stl_file_name="Chassi_top.stl" z="0.03"/>
 <xacro:add_base_plate name="lower_plate" stl_file_name="Chassi_bottom.stl" z="-0.03"/>
+<xacro:if value="$(arg use_gazebo_simulation)">
 <gazebo>
   <plugin filename="libgazebo_ros2_control.so" name="gazebo_ros2_control" >
     <parameters>$(find penta_description)/config/ros2_control_params.yaml</parameters>
   </plugin>
+  <xacro:include filename="$(find penta_description)/ros2_control/gazebo.ros2_control.xacro" />
 </gazebo>
-<xacro:include filename="$(find penta_description)/ros2_control/pca9685.ros2_control.xacro">
+</xacro:if>
+<xacro:if value="$(arg use_pca9685_ros2_control)">
+  <xacro:include filename="$(find penta_description)/ros2_control/pca9685.ros2_control.xacro" />
   <xacro:add_pca9685_hw_interface name="pca9685" prefix="penta_" use_mock_hardware="false"/>
-</xacro:include>
+</xacro:if>
 </robot>

File: penta_description/urdf/single_limb.urdf.xacro (robot description, xacro)
@@ -1,5 +1,5 @@
 <?xml version="1.0"?>
 <robot xmlns:xacro="http://www.ros.org/wiki/xacro">
-  <xacro:macro name="add_leg" params="prefix shoulderxyz shoulderrpy">
+  <xacro:macro name="add_leg" params="prefix shoulderxyz shoulderrpy use_gazebo_simulation">
     <link name="${prefix}_shoulder_motor">
       <visual>
@@ -133,4 +133,5 @@
       <origin xyz="0.0 0.0 0.0" rpy="0 0 0"/>
     </joint>
+  <xacro:if value="${use_gazebo_simulation}">
     <!-- ros2_control interfaces for each joint -->
     <ros2_control name="${prefix}_ros2_control" type="system">
@@ -185,4 +186,5 @@
       </actuator>
     </transmission>
+  </xacro:if>
   </xacro:macro>
 </robot>
