Commit message: add name space into xacro and inside nodes

File: penta_description/urdf/penta.urdf.xacro (robot description, xacro)
@@ -1,4 +1,5 @@
 <?xml version="1.0"?>
 <robot name="penta_bot" xmlns:xacro="http://www.ros.org/wiki/xacro">
+  <xacro:arg name="name_space" default="" />
   <xacro:arg name="use_gazebo_simulation" default="False" />
   <xacro:arg name="use_pca9685_ros2_control" default="False" />
@@ -56,6 +57,6 @@
     <origin xyz="-0.1 0.0 0.025" rpy="0 0 0"/>
   </joint>
-  <xacro:macro name="add_base_plate" params="name stl_file_name z">
-    <link name="${name}_link">
+  <xacro:macro name="add_base_plate" params="name_space name stl_file_name z">
+    <link name="${name_space}${name}_link">
       <visual>
         <geometry>
@@ -66,17 +67,17 @@
       </visual>
     </link>
-    <joint name="${name}_joint" type="fixed">
+    <joint name="${name_space}${name}_joint" type="fixed">
       <parent link="base_link"/>
-      <child link="${name}_link"/>
+      <child link="${name_space}${name}_link"/>
     <origin xyz="0.0 0.0 ${z}" rpy="0 0 0"/>
   </joint>
   </xacro:macro>
-<xacro:add_leg prefix="limb0" shoulderxyz="${0.085*cos(0.*3.141592/2.5)} ${0.085*sin(0.*3.141592/2.5)} 0." shoulderrpy="0. 0. ${(0.*3.141592/2.5)}" use_gazebo_simulation="$(arg use_gazebo_simulation)"/>
-<xacro:add_leg prefix="limb1" shoulderxyz="${0.085*cos(1.*3.141592/2.5)} ${0.085*sin(1.*3.141592/2.5)} 0." shoulderrpy="0. 0. ${(1.*3.141592/2.5)}" use_gazebo_simulation="$(arg use_gazebo_simulation)"/>
-<xacro:add_leg prefix="limb2" shoulderxyz="${0.085*cos(2.*3.141592/2.5)} ${0.085*sin(2.*3.141592/2.5)} 0." shoulderrpy="0. 0. ${(2.*3.141592/2.5)}" use_gazebo_simulation="$(arg use_gazebo_simulation)"/>
-<xacro:add_leg prefix="limb3" shoulderxyz="${0.085*cos(3.*3.141592/2.5)} ${0.085*sin(3.*3.141592/2.5)} 0." shoulderrpy="0. 0. ${(3.*3.141592/2.5)}" use_gazebo_simulation="$(arg use_gazebo_simulation)"/>
-<xacro:add_leg prefix="limb4" shoulderxyz="${0.085*cos(4.*3.141592/2.5)} ${0.085*sin(4.*3.141592/2.5)} 0." shoulderrpy="0. 0. ${(4.*3.141592/2.5)}" use_gazebo_simulation="$(arg use_gazebo_simulation)"/>
-<xacro:add_base_plate name="upper_plate" stl_file_name="Chassi_top.stl" z="0.03"/>
-<xacro:add_base_plate name="lower_plate" stl_file_name="Chassi_bottom.stl" z="-0.03"/>
+<xacro:add_leg name_space="$(arg name_space)" prefix="limb0" shoulderxyz="${0.085*cos(0.*3.141592/2.5)} ${0.085*sin(0.*3.141592/2.5)} 0." shoulderrpy="0. 0. ${(0.*3.141592/2.5)}" use_gazebo_simulation="$(arg use_gazebo_simulation)"/>
+<xacro:add_leg name_space="$(arg name_space)" prefix="limb1" shoulderxyz="${0.085*cos(1.*3.141592/2.5)} ${0.085*sin(1.*3.141592/2.5)} 0." shoulderrpy="0. 0. ${(1.*3.141592/2.5)}" use_gazebo_simulation="$(arg use_gazebo_simulation)"/>
+<xacro:add_leg name_space="$(arg name_space)" prefix="limb2" shoulderxyz="${0.085*cos(2.*3.141592/2.5)} ${0.085*sin(2.*3.141592/2.5)} 0." shoulderrpy="0. 0. ${(2.*3.141592/2.5)}" use_gazebo_simulation="$(arg use_gazebo_simulation)"/>
+<xacro:add_leg name_space="$(arg name_space)" prefix="limb3" shoulderxyz="${0.085*cos(3.*3.141592/2.5)} ${0.085*sin(3.*3.141592/2.5)} 0." shoulderrpy="0. 0. ${(3.*3.141592/2.5)}" use_gazebo_simulation="$(arg use_gazebo_simulation)"/>
+<xacro:add_leg name_space="$(arg name_space)" prefix="limb4" shoulderxyz="${0.085*cos(4.*3.141592/2.5)} ${0.085*sin(4.*3.141592/2.5)} 0." shoulderrpy="0. 0. ${(4.*3.141592/2.5)}" use_gazebo_simulation="$(arg use_gazebo_simulation)"/>
+<xacro:add_base_plate name_space="$(arg name_space)" name="upper_plate" stl_file_name="Chassi_top.stl" z="0.03"/>
+<xacro:add_base_plate name_space="$(arg name_space)" name="lower_plate" stl_file_name="Chassi_bottom.stl" z="-0.03"/>
 <xacro:if value="$(arg use_gazebo_simulation)">
 <gazebo>
@@ -89,5 +90,5 @@
 <xacro:if value="$(arg use_pca9685_ros2_control)">
   <xacro:include filename="$(find penta_description)/ros2_control/pca9685.ros2_control.xacro" />
-  <xacro:add_pca9685_hw_interface name="pca9685" prefix="penta_" use_mock_hardware="false"/>
+  <xacro:add_pca9685_hw_interface name="pca9685" prefix="$(arg name_space)" use_mock_hardware="false"/>
 </xacro:if>
 </robot>

File: penta_description/urdf/single_limb.urdf.xacro (robot description, xacro)
@@ -1,6 +1,6 @@
 <?xml version="1.0"?>
 <robot xmlns:xacro="http://www.ros.org/wiki/xacro">
-  <xacro:macro name="add_leg" params="prefix shoulderxyz shoulderrpy use_gazebo_simulation">
-    <link name="${prefix}_shoulder_motor">
+  <xacro:macro name="add_leg" params="name_space prefix shoulderxyz shoulderrpy use_gazebo_simulation">
+    <link name="${name_space}${prefix}_shoulder_motor">
       <visual>
         <geometry>
@@ -16,5 +16,5 @@
       </inertial>
     </link>
-    <link name="${prefix}_shoulder_link">
+    <link name="${name_space}${prefix}_shoulder_link">
       <visual>
         <geometry>
@@ -30,5 +30,5 @@
       </inertial>
     </link>
-    <link name="${prefix}_upper_arm_link">
+    <link name="${name_space}${prefix}_upper_arm_link">
       <visual>
         <geometry>
@@ -44,5 +44,5 @@
       </inertial>
     </link>
-    <link name="${prefix}_lower_arm_link">
+    <link name="${name_space}${prefix}_lower_arm_link">
       <visual>
         <geometry>
@@ -58,5 +58,5 @@
       </inertial>
     </link>
-    <link name="${prefix}_foot">
+    <link name="${name_space}${prefix}_foot">
       <visual>
         <geometry>
@@ -105,49 +105,49 @@
       </collision>
     </link>
-    <joint name="${prefix}/joint_shoulder_motor" type="fixed">
+    <joint name="${name_space}${prefix}/joint_shoulder_motor" type="fixed">
       <parent link="base_link"/>
-      <child link="${prefix}_shoulder_motor"/>
+      <child link="${name_space}${prefix}_shoulder_motor"/>
       <origin xyz="${shoulderxyz}" rpy="${shoulderrpy}"/>
     </joint>
-    <joint name="${prefix}/joint0" type="continuous">
-      <parent link="${prefix}_shoulder_motor"/>
-      <child link="${prefix}_shoulder_link"/>
+    <joint name="${name_space}${prefix}/joint0" type="continuous">
+      <parent link="${name_space}${prefix}_shoulder_motor"/>
+      <child link="${name_space}${prefix}_shoulder_link"/>
       <origin xyz="0.0 0.0 0.0" rpy="0 0 0"/>
       <axis xyz="0 0 1" />
     </joint>
-    <joint name="${prefix}/joint1" type="continuous">
-      <parent link="${prefix}_shoulder_link"/>
-      <child link="${prefix}_upper_arm_link"/>
+    <joint name="${name_space}${prefix}/joint1" type="continuous">
+      <parent link="${name_space}${prefix}_shoulder_link"/>
+      <child link="${name_space}${prefix}_upper_arm_link"/>
       <origin xyz="0.0455 0.0 0.0" rpy="-1.57 0 0"/>
       <axis xyz="0 0 1" />
     </joint>
-    <joint name="${prefix}/joint2" type="continuous">
-      <parent link="${prefix}_upper_arm_link"/>
-      <child link="${prefix}_lower_arm_link"/>
+    <joint name="${name_space}${prefix}/joint2" type="continuous">
+      <parent link="${name_space}${prefix}_upper_arm_link"/>
+      <child link="${name_space}${prefix}_lower_arm_link"/>
       <origin xyz="0.096 0.0 0.0" rpy="0 0 0"/>
       <axis xyz="0 0 1" />
     </joint>
-    <joint name="${prefix}/joint3" type="fixed">
-      <parent link="${prefix}_lower_arm_link"/>
-      <child link="${prefix}_foot"/>
+    <joint name="${name_space}${prefix}/joint3" type="fixed">
+      <parent link="${name_space}${prefix}_lower_arm_link"/>
+      <child link="${name_space}${prefix}_foot"/>
       <origin xyz="0.0 0.0 0.0" rpy="0 0 0"/>
     </joint>
   <xacro:if value="${use_gazebo_simulation}">
     <!-- ros2_control interfaces for each joint -->
-    <ros2_control name="${prefix}_ros2_control" type="system">
+    <ros2_control name="${name_space}${prefix}_ros2_control" type="system">
       <hardware>
         <plugin>gazebo_ros2_control/GazeboSystem</plugin>
       </hardware>
-      <joint name="${prefix}/joint0">
+      <joint name="${name_space}${prefix}/joint0">
         <command_interface name="position"/>
         <state_interface name="position"/>
         <state_interface name="velocity"/>
       </joint>
-      <joint name="${prefix}/joint1">
+      <joint name="${name_space}${prefix}/joint1">
         <command_interface name="position"/>
         <state_interface name="position"/>
         <state_interface name="velocity"/>
       </joint>
-      <joint name="${prefix}/joint2">
+      <joint name="${name_space}${prefix}/joint2">
         <command_interface name="position"/>
         <state_interface name="position"/>
@@ -156,30 +156,30 @@
     </ros2_control>
     <!-- Transmission blocks -->
-    <transmission name="${prefix}_joint0_trans">
+    <transmission name="${name_space}${prefix}_joint0_trans">
       <type>transmission_interface/SimpleTransmission</type>
-      <joint name="${prefix}/joint0">
+      <joint name="${name_space}${prefix}/joint0">
         <hardwareInterface>hardware_interface/PositionJointInterface</hardwareInterface>
       </joint>
-      <actuator name="${prefix}_motor0">
+      <actuator name="${name_space}${prefix}_motor0">
         <hardwareInterface>hardware_interface/PositionJointInterface</hardwareInterface>
         <mechanicalReduction>1</mechanicalReduction>
       </actuator>
     </transmission>
-    <transmission name="${prefix}_joint1_trans">
+    <transmission name="${name_space}${prefix}_joint1_trans">
       <type>transmission_interface/SimpleTransmission</type>
-      <joint name="${prefix}/joint1">
+      <joint name="${name_space}${prefix}/joint1">
         <hardwareInterface>hardware_interface/PositionJointInterface</hardwareInterface>
       </joint>
-      <actuator name="${prefix}_motor1">
+      <actuator name="${name_space}${prefix}_motor1">
         <hardwareInterface>hardware_interface/PositionJointInterface</hardwareInterface>
         <mechanicalReduction>1</mechanicalReduction>
       </actuator>
     </transmission>
-    <transmission name="${prefix}_joint2_trans">
+    <transmission name="${name_space}${prefix}_joint2_trans">
       <type>transmission_interface/SimpleTransmission</type>
-      <joint name="${prefix}/joint2">
+      <joint name="${name_space}${prefix}/joint2">
         <hardwareInterface>hardware_interface/PositionJointInterface</hardwareInterface>
       </joint>
-      <actuator name="${prefix}_motor2">
+      <actuator name="${name_space}${prefix}_motor2">
         <hardwareInterface>hardware_interface/PositionJointInterface</hardwareInterface>
         <mechanicalReduction>1</mechanicalReduction>

Commit message: add name spaces to allow simulating several robots with different name space

File: penta_description/urdf/penta.urdf.xacro (robot description, xacro)
@@ -18,6 +18,7 @@
       </material>
   </xacro:macro>
-  <link name="base_footprint"/>
-  <link name="base_link">
+<xacro:macro name="add_body" params="name_space">
+  <link name="${name_space}base_footprint"/>
+  <link name="${name_space}base_link">
     <visual>
       <geometry>
@@ -39,10 +40,10 @@
     </inertial>
   </link>
-  <joint name="joint_robot_body_center" type="fixed">
-    <parent link="base_footprint"/>
-    <child link="base_link"/>
+  <joint name="${name_space}joint_robot_body_center" type="fixed">
+    <parent link="${name_space}base_footprint"/>
+    <child link="${name_space}base_link"/>
     <origin xyz="0.0 0.0 0.075" rpy="0 0 0"/>
   </joint>
-  <link name="head_link">
+  <link name="${name_space}head_link">
     <visual>
       <geometry>
@@ -52,9 +53,10 @@
     </visual>
   </link>
-  <joint name="head_base" type="fixed">
-    <parent link="base_link"/>
-    <child link="head_link"/>
+  <joint name="${name_space}head_base" type="fixed">
+    <parent link="${name_space}base_link"/>
+    <child link="${name_space}head_link"/>
     <origin xyz="-0.1 0.0 0.025" rpy="0 0 0"/>
   </joint>
+</xacro:macro>
   <xacro:macro name="add_base_plate" params="name_space name stl_file_name z">
     <link name="${name_space}${name}_link">
@@ -68,9 +70,10 @@
     </link>
     <joint name="${name_space}${name}_joint" type="fixed">
-      <parent link="base_link"/>
+      <parent link="${name_space}base_link"/>
       <child link="${name_space}${name}_link"/>
     <origin xyz="0.0 0.0 ${z}" rpy="0 0 0"/>
   </joint>
   </xacro:macro>
+<xacro:add_body name_space="$(arg name_space)"/>
 <xacro:add_leg name_space="$(arg name_space)" prefix="limb0" shoulderxyz="${0.085*cos(0.*3.141592/2.5)} ${0.085*sin(0.*3.141592/2.5)} 0." shoulderrpy="0. 0. ${(0.*3.141592/2.5)}" use_gazebo_simulation="$(arg use_gazebo_simulation)"/>
 <xacro:add_leg name_space="$(arg name_space)" prefix="limb1" shoulderxyz="${0.085*cos(1.*3.141592/2.5)} ${0.085*sin(1.*3.141592/2.5)} 0." shoulderrpy="0. 0. ${(1.*3.141592/2.5)}" use_gazebo_simulation="$(arg use_gazebo_simulation)"/>

File: penta_description/urdf/single_limb.urdf.xacro (robot description, xacro)
@@ -106,5 +106,5 @@
     </link>
     <joint name="${name_space}${prefix}/joint_shoulder_motor" type="fixed">
-      <parent link="base_link"/>
+      <parent link="${name_space}base_link"/>
       <child link="${name_space}${prefix}_shoulder_motor"/>
       <origin xyz="${shoulderxyz}" rpy="${shoulderrpy}"/>

Commit message: wip: fix urdf after merge with fix_name_space

File: penta_description/urdf/penta.urdf.xacro (robot description, xacro)
@@ -1,6 +1,9 @@
 <?xml version="1.0"?>
 <robot name="penta_bot" xmlns:xacro="http://www.ros.org/wiki/xacro">
+  <xacro:arg name="name_space" default="" />
+  <xacro:arg name="use_gazebo_simulation" default="False" />
+  <xacro:arg name="use_pca9685_ros2_control" default="False" />
   <xacro:include filename="$(find penta_description)/urdf/penta_robot_macro.urdf.xacro" />
-  <xacro:add_penta_bot/>
+  <xacro:add_penta_bot name_space="$(arg name_space)" use_gazebo_simulation="$(arg use_gazebo_simulation)" use_pca9685_ros2_control="$(arg use_pca9685_ros2_control)"/>
   <!-- gazebo ros2_control plugins -->
   <gazebo>

File: penta_description/urdf/penta_robot_macro.urdf.xacro (robot description, xacro)
@@ -1,5 +1,5 @@
 <?xml version="1.0"?>
 <robot xmlns:xacro="http://www.ros.org/wiki/xacro">
-  <xacro:macro name="add_penta_bot">
+  <xacro:macro name="add_penta_bot" params="name_space use_gazebo_simulation use_pca9685_ros2_control">
     <xacro:property name="PI" value="3.141592" />
     <xacro:property name="PI2" value="${PI/2}" />
@@ -71,9 +71,9 @@
     </joint>
     </xacro:macro>
-    <xacro:add_leg prefix="limb0" shoulderxyz="${0.085*cos(0.*3.141592/2.5)} ${0.085*sin(0.*3.141592/2.5)} 0." shoulderrpy="0. 0. ${(0.*3.141592/2.5)}"/>
-    <xacro:add_leg prefix="limb1" shoulderxyz="${0.085*cos(1.*3.141592/2.5)} ${0.085*sin(1.*3.141592/2.5)} 0." shoulderrpy="0. 0. ${(1.*3.141592/2.5)}"/>
-    <xacro:add_leg prefix="limb2" shoulderxyz="${0.085*cos(2.*3.141592/2.5)} ${0.085*sin(2.*3.141592/2.5)} 0." shoulderrpy="0. 0. ${(2.*3.141592/2.5)}"/>
-    <xacro:add_leg prefix="limb3" shoulderxyz="${0.085*cos(3.*3.141592/2.5)} ${0.085*sin(3.*3.141592/2.5)} 0." shoulderrpy="0. 0. ${(3.*3.141592/2.5)}"/>
-    <xacro:add_leg prefix="limb4" shoulderxyz="${0.085*cos(4.*3.141592/2.5)} ${0.085*sin(4.*3.141592/2.5)} 0." shoulderrpy="0. 0. ${(4.*3.141592/2.5)}"/>
+    <xacro:add_leg prefix="limb0" shoulderxyz="${0.085*cos(0.*3.141592/2.5)} ${0.085*sin(0.*3.141592/2.5)} 0." shoulderrpy="0. 0. ${(0.*3.141592/2.5)}" name_space="${name_space}" use_gazebo_simulation="${use_gazebo_simulation}"/>
+    <xacro:add_leg prefix="limb1" shoulderxyz="${0.085*cos(1.*3.141592/2.5)} ${0.085*sin(1.*3.141592/2.5)} 0." shoulderrpy="0. 0. ${(1.*3.141592/2.5)}" name_space="${name_space}" use_gazebo_simulation="${use_gazebo_simulation}"/>
+    <xacro:add_leg prefix="limb2" shoulderxyz="${0.085*cos(2.*3.141592/2.5)} ${0.085*sin(2.*3.141592/2.5)} 0." shoulderrpy="0. 0. ${(2.*3.141592/2.5)}" name_space="${name_space}" use_gazebo_simulation="${use_gazebo_simulation}"/>
+    <xacro:add_leg prefix="limb3" shoulderxyz="${0.085*cos(3.*3.141592/2.5)} ${0.085*sin(3.*3.141592/2.5)} 0." shoulderrpy="0. 0. ${(3.*3.141592/2.5)}" name_space="${name_space}" use_gazebo_simulation="${use_gazebo_simulation}"/>
+    <xacro:add_leg prefix="limb4" shoulderxyz="${0.085*cos(4.*3.141592/2.5)} ${0.085*sin(4.*3.141592/2.5)} 0." shoulderrpy="0. 0. ${(4.*3.141592/2.5)}" name_space="${name_space}" use_gazebo_simulation="${use_gazebo_simulation}"/>
     <xacro:add_base_plate name="upper_plate" stl_file_name="Chassi_top.stl" z="0.03"/>
     <xacro:add_base_plate name="lower_plate" stl_file_name="Chassi_bottom.stl" z="-0.03"/>
