Commit message: fix name spaces

File: penta_description/urdf/lidar.urdf.xacro (robot description, xacro)
@@ -16,5 +16,5 @@
       </inertial>
     </link>
-    <joint name="${name_space}/${name_space}laser_joint" type="fixed">
+    <joint name="laser_joint" type="fixed">
       <parent link="${name_space}base_link"/>
       <child link="${name_space}laser_frame"/>

File: penta_description/urdf/penta_robot_macro.urdf.xacro (robot description, xacro)
@@ -43,5 +43,5 @@
       </inertial>
     </link>
-    <joint name="${name_space}joint_robot_body_center" type="fixed">
+    <joint name="joint_robot_body_center" type="fixed">
       <parent link="${name_space}base_footprint"/>
       <child link="${name_space}base_link"/>
@@ -56,5 +56,5 @@
       </visual>
     </link>
-    <joint name="${name_space}head_base" type="fixed">
+    <joint name="head_base" type="fixed">
       <parent link="${name_space}base_link"/>
       <child link="${name_space}head_link"/>

File: penta_description/urdf/single_limb.urdf.xacro (robot description, xacro)
@@ -105,10 +105,10 @@
       </collision>
     </link>
-    <joint name="${name_space}${prefix}/joint_shoulder_motor" type="fixed">
+    <joint name="${prefix}/joint_shoulder_motor" type="fixed">
       <parent link="${name_space}base_link"/>
       <child link="${name_space}${prefix}_shoulder_motor"/>
       <origin xyz="${shoulderxyz}" rpy="${shoulderrpy}"/>
     </joint>
-    <joint name="${name_space}${prefix}/joint0" type="continuous">
+    <joint name="${prefix}/joint0" type="continuous">
       <parent link="${name_space}${prefix}_shoulder_motor"/>
       <child link="${name_space}${prefix}_shoulder_link"/>
@@ -116,5 +116,5 @@
       <axis xyz="0 0 1" />
     </joint>
-    <joint name="${name_space}${prefix}/joint1" type="continuous">
+    <joint name="${prefix}/joint1" type="continuous">
       <parent link="${name_space}${prefix}_shoulder_link"/>
       <child link="${name_space}${prefix}_upper_arm_link"/>
@@ -122,5 +122,5 @@
       <axis xyz="0 0 1" />
     </joint>
-    <joint name="${name_space}${prefix}/joint2" type="continuous">
+    <joint name="${prefix}/joint2" type="continuous">
       <parent link="${name_space}${prefix}_upper_arm_link"/>
       <child link="${name_space}${prefix}_lower_arm_link"/>
@@ -128,5 +128,5 @@
       <axis xyz="0 0 1" />
     </joint>
-    <joint name="${name_space}${prefix}/joint3" type="fixed">
+    <joint name="${prefix}/joint3" type="fixed">
       <parent link="${name_space}${prefix}_lower_arm_link"/>
       <child link="${name_space}${prefix}_foot"/>
@@ -139,5 +139,5 @@
         <plugin>gz_ros2_control/GazeboSimSystem</plugin>
       </hardware>
-      <joint name="${name_space}${prefix}/joint0">
+      <joint name="${prefix}/joint0">
         <command_interface name="position"/>
         <state_interface name="position">
@@ -146,5 +146,5 @@
         <state_interface name="velocity"/>
       </joint>
-      <joint name="${name_space}${prefix}/joint1">
+      <joint name="${prefix}/joint1">
         <command_interface name="position"/>
         <state_interface name="position">
@@ -153,5 +153,5 @@
         <state_interface name="velocity"/>
       </joint>
-      <joint name="${name_space}${prefix}/joint2">
+      <joint name="${prefix}/joint2">
         <command_interface name="position"/>
         <state_interface name="position">
@@ -162,30 +162,30 @@
     </ros2_control>
     <!-- Transmission blocks -->
-    <transmission name="${name_space}${prefix}_joint0_trans">
+    <transmission name="${prefix}_joint0_trans">
       <type>transmission_interface/SimpleTransmission</type>
-      <joint name="${name_space}${prefix}/joint0">
+      <joint name="${prefix}/joint0">
         <hardwareInterface>hardware_interface/PositionJointInterface</hardwareInterface>
       </joint>
-      <actuator name="${name_space}${prefix}_motor0">
+      <actuator name="${prefix}_motor0">
         <hardwareInterface>hardware_interface/PositionJointInterface</hardwareInterface>
         <mechanicalReduction>1</mechanicalReduction>
       </actuator>
     </transmission>
-    <transmission name="${name_space}${prefix}_joint1_trans">
+    <transmission name="${prefix}_joint1_trans">
       <type>transmission_interface/SimpleTransmission</type>
-      <joint name="${name_space}${prefix}/joint1">
+      <joint name="${prefix}/joint1">
         <hardwareInterface>hardware_interface/PositionJointInterface</hardwareInterface>
       </joint>
-      <actuator name="${name_space}${prefix}_motor1">
+      <actuator name="${prefix}_motor1">
         <hardwareInterface>hardware_interface/PositionJointInterface</hardwareInterface>
         <mechanicalReduction>1</mechanicalReduction>
       </actuator>
     </transmission>
-    <transmission name="${name_space}${prefix}_joint2_trans">
+    <transmission name="${prefix}_joint2_trans">
       <type>transmission_interface/SimpleTransmission</type>
-      <joint name="${name_space}${prefix}/joint2">
+      <joint name="${prefix}/joint2">
         <hardwareInterface>hardware_interface/PositionJointInterface</hardwareInterface>
       </joint>
-      <actuator name="${name_space}${prefix}_motor2">
+      <actuator name="${prefix}_motor2">
         <hardwareInterface>hardware_interface/PositionJointInterface</hardwareInterface>
         <mechanicalReduction>1</mechanicalReduction>
